File: DYNAMO-PCB/DYNAMO-PCB.kicad_sch (KiCad schematic)
At the start: 18 parts

Commit message: further simplified
Parts:
- removed Camera1, Camera2, Microphone1, Microphone2, Misc1, Misc2: USB3_A, 692122030100:692122030100, symbol Connector:USB3_A
- removed Display_A1, Display_A2, Display_B1, Display_B2: HDMI_A, Connector_Video:HDMI_A_Molex_208658-1001_Horizontal, symbol Connector:HDMI_A
- removed Speaker1, Speaker2: SJ1-3533NS, SJ1-3533NS:CUI_SJ1-3533NS, symbol SJ1-3533NS:SJ1-3533NS
Connections:
- no-connect marks 86 -> 82
Other:
- moved on the sheet: A1A, A1B, C1, HeadFlat1, R1
