File: DYNAMO-PCB/powerdistrib.kicad_sch (KiCad schematic)
At the start: 13 parts, among them J14 USB_C_Receptacle_PowerOnly_6P, J15 USB_C_Receptacle_PowerOnly_6P, J17 USB3_A, J19 USB3_A, J2 USB3_A, J26 USB_C_Receptacle_PowerOnly_6P, J28 USB_C_Receptacle_PowerOnly_6P, J31 USB3_A, J32 USB3_A, J4 USB_C_Receptacle_PowerOnly_6P

Commit message: routing
Parts:
- renumbered J17 to DisplayPWR1, J2 to DisplayPWR2, J26 to MainPWR1, J28 to MainPWR2, J32 to Modem1, J31 to ModemPWR1, S2 to ON/OFFmain1, S3 to ON/OFFmodem1, S1 to ON/OFFperipherals1, J19 to PeripheralsPWR1, J4 to RechargeA1, J14 to RechargeB1, J15 to RechargeB2
Changed lines of the file:
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@@
 	(text_box "4G modem port"
 		(exclude_from_sim no)
-		(at 110.49 125.73 0)
+		(at 113.03 125.73 0)
 		(size 80.01 41.91)
 		(margins 0.9525 0.9525 0.9525 0.9525)
@@
 		(on_board yes)
 		(dnp no)
-		(property "Reference" "J15"
+		(property "Reference" "RechargeB2"
 			(at 66.04 118.11 0)
 			(effects
@@
 			(project "DYNAMO-PCB"
 				(path "/2ca9dd43-411d-4cc5-8a4b-ed00d72bae91/b1a71f53-bc17-4314-9292-b5c15f4aa94b"
-					(reference "J15")
+					(reference "RechargeB2")
 					(unit 1)
 				)
@@
 		(dnp no)
 		(fields_autoplaced yes)
-		(property "Reference" "J26"
+		(property "Reference" "MainPWR1"
 			(at 127 66.04 0)
 			(effects
@@
 			(project "DYNAMO-PCB"
 				(path "/2ca9dd43-411d-4cc5-8a4b-ed00d72bae91/b1a71f53-bc17-4314-9292-b5c15f4aa94b"
-					(reference "J26")
+					(reference "MainPWR1")
 					(unit 1)
 				)
@@
 		(dnp no)
 		(fields_autoplaced yes)
-		(property "Reference" "J14"
+		(property "Reference" "RechargeB1"
 			(at 31.75 118.11 0)
 			(effects
@@
 			(project "DYNAMO-PCB"
 				(path "/2ca9dd43-411d-4cc5-8a4b-ed00d72bae91/b1a71f53-bc17-4314-9292-b5c15f4aa94b"
-					(reference "J14")
+					(reference "RechargeB1")
 					(unit 1)
 				)
@@
 		(on_board yes)
 		(dnp no)
-		(property "Reference" "J31"
-			(at 124.46 124.46 0)
+		(property "Reference" "ModemPWR1"
+			(at 124.46 130.81 0)
 			(effects
 				(font
@@
 			(project "DYNAMO-PCB"
 				(path "/2ca9dd43-411d-4cc5-8a4b-ed00d72bae91/b1a71f53-bc17-4314-9292-b5c15f4aa94b"
-					(reference "J31")
+					(reference "ModemPWR1")
 					(unit 1)
 				)
@@
 		(dnp no)
 		(fields_autoplaced yes)
-		(property "Reference" "J4"
+		(property "Reference" "RechargeA1"
 			(at 30.48 78.74 0)
 			(effects
@@
 			(project ""
 				(path "/2ca9dd43-411d-4cc5-8a4b-ed00d72bae91/b1a71f53-bc17-4314-9292-b5c15f4aa94b"
-					(reference "J4")
+					(reference "RechargeA1")
 					(unit 1)
 				)
@@
 		(on_board yes)
 		(dnp no)
-		(property "Reference" "S1"
+		(property "Reference" "ON/OFFperipherals1"
 			(at 227.33 80.01 0)
 			(effects
@@
 			(project "DYNAMO-PCB"
 				(path "/2ca9dd43-411d-4cc5-8a4b-ed00d72bae91/b1a71f53-bc17-4314-9292-b5c15f4aa94b"
-					(reference "S1")
+					(reference "ON/OFFperipherals1")
 					(unit 1)
 				)
@@
 		(on_board yes)
 		(dnp no)
-		(property "Reference" "S3"
+		(property "Reference" "ON/OFFmodem1"
 			(at 151.13 135.89 0)
 			(effects
@@
 			(project "DYNAMO-PCB"
 				(path "/2ca9dd43-411d-4cc5-8a4b-ed00d72bae91/b1a71f53-bc17-4314-9292-b5c15f4aa94b"
-					(reference "S3")
+					(reference "ON/OFFmodem1")
 					(unit 1)
 				)
@@
 		(on_board yes)
 		(dnp no)
-		(property "Reference" "J32"
-			(at 177.8 124.46 0)
+		(property "Reference" "Modem1"
+			(at 177.8 130.81 0)
 			(effects
 				(font
@@
 			(project "DYNAMO-PCB"
 				(path "/2ca9dd43-411d-4cc5-8a4b-ed00d72bae91/b1a71f53-bc17-4314-9292-b5c15f4aa94b"
-					(reference "J32")
+					(reference "Modem1")
 					(unit 1)
 				)
@@
 		(on_board yes)
 		(dnp no)
-		(property "Reference" "J19"
+		(property "Reference" "PeripheralsPWR1"
 			(at 205.74 68.58 0)
 			(effects
@@
 			(project "DYNAMO-PCB"
 				(path "/2ca9dd43-411d-4cc5-8a4b-ed00d72bae91/b1a71f53-bc17-4314-9292-b5c15f4aa94b"
-					(reference "J19")
+					(reference "PeripheralsPWR1")
 					(unit 1)
 				)
@@
 		(on_board yes)
 		(dnp no)
-		(property "Reference" "J28"
+		(property "Reference" "MainPWR2"
 			(at 175.26 66.04 0)
 			(effects
@@
 			(project "DYNAMO-PCB"
 				(path "/2ca9dd43-411d-4cc5-8a4b-ed00d72bae91/b1a71f53-bc17-4314-9292-b5c15f4aa94b"
-					(reference "J28")
+					(reference "MainPWR2")
 					(unit 1)
 				)
@@
 		(dnp no)
 		(fields_autoplaced yes)
-		(property "Reference" "J17"
+		(property "Reference" "DisplayPWR1"
 			(at 237.49 33.0199 90)
 			(effects
@@
 			(project "DYNAMO-PCB"
 				(path "/2ca9dd43-411d-4cc5-8a4b-ed00d72bae91/b1a71f53-bc17-4314-9292-b5c15f4aa94b"
-					(reference "J17")
+					(reference "DisplayPWR1")
 					(unit 1)
 				)
@@
 		(on_board yes)
 		(dnp no)
-		(property "Reference" "J2"
+		(property "Reference" "DisplayPWR2"
 			(at 240.03 33.0199 90)
 			(effects
@@
 			(project "DYNAMO-PCB"
 				(path "/2ca9dd43-411d-4cc5-8a4b-ed00d72bae91/b1a71f53-bc17-4314-9292-b5c15f4aa94b"
-					(reference "J2")
+					(reference "DisplayPWR2")
 					(unit 1)
 				)
@@
 		(dnp no)
 		(fields_autoplaced yes)
-		(property "Reference" "S2"
+		(property "Reference" "ON/OFFmain1"
 			(at 151.13 68.58 0)
 			(effects
@@
 			(project "DYNAMO-PCB"
 				(path "/2ca9dd43-411d-4cc5-8a4b-ed00d72bae91/b1a71f53-bc17-4314-9292-b5c15f4aa94b"
-					(reference "S2")
+					(reference "ON/OFFmain1")
 					(unit 1)
 				)

Commit message: further simplified
Changed lines of the file:
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@@
 	(text_box "Lattepanda powering"
 		(exclude_from_sim no)
-		(at 110.49 63.5 0)
+		(at 110.49 62.23 0)
 		(size 78.74 49.53)
 		(margins 0.9525 0.9525 0.9525 0.9525)
@@
 	)
 	(junction
-		(at 142.24 88.9)
+		(at 147.32 88.9)
 		(diameter 0)
 		(color 0 0 0 0)
@@
 	)
 	(junction
-		(at 142.24 91.44)
+		(at 146.05 91.44)
 		(diameter 0)
 		(color 0 0 0 0)
@@
 	(wire
 		(pts
-			(xy 147.32 71.12) (xy 147.32 83.82)
-		)
-		(stroke
-			(width 0)
-			(type default)
-		)
-	)
-	(wire
-		(pts
-			(xy 146.05 72.39) (xy 146.05 87.63)
+			(xy 147.32 71.12) (xy 147.32 88.9)
+		)
+		(stroke
+			(width 0)
+			(type default)
+		)
+	)
+	(wire
+		(pts
+			(xy 146.05 72.39) (xy 146.05 91.44)
 		)
 		(stroke
@@
 	(wire
 		(pts
-			(xy 142.24 88.9) (xy 160.02 88.9)
+			(xy 147.32 88.9) (xy 160.02 88.9)
 		)
 		(stroke
@@
 	(wire
 		(pts
-			(xy 146.05 87.63) (xy 142.24 91.44)
-		)
-		(stroke
-			(width 0)
-			(type default)
-		)
-	)
-	(wire
-		(pts
 			(xy 222.25 55.88) (xy 222.25 105.41)
 		)
@@
 	(wire
 		(pts
+			(xy 146.05 91.44) (xy 142.24 91.44)
+		)
+		(stroke
+			(width 0)
+			(type default)
+		)
+	)
+	(wire
+		(pts
 			(xy 134.62 58.42) (xy 147.32 71.12)
 		)
@@
 	(wire
 		(pts
+			(xy 147.32 88.9) (xy 142.24 88.9)
+		)
+		(stroke
+			(width 0)
+			(type default)
+		)
+	)
+	(wire
+		(pts
 			(xy 46.99 140.97) (xy 50.8 140.97)
 		)
@@
 	(wire
 		(pts
-			(xy 142.24 91.44) (xy 160.02 91.44)
+			(xy 146.05 91.44) (xy 160.02 91.44)
 		)
 		(stroke
@@
 		)
 		(stroke
-			(width 0)
-			(type default)
-		)
-	)
-	(wire
-		(pts
-			(xy 147.32 83.82) (xy 142.24 88.9)
-		)
-		(stroke
