File: DYNAMO-PCB/DYNAMO-PCB.kicad_pcb (KiCad board)
At the start: 2 copper layers, 42 parts, among them J10 Conn_01x03_Pin, J11 Conn_01x03_Pin, J12 Conn_01x03_Pin, J13 Conn_01x02_Pin, J14 USB_C_Receptacle_PowerOnly_6P, J15 USB_C_Receptacle_PowerOnly_6P, J17 USB3_A, J18 USB3_A, J19 USB3_A, J2 USB3_A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

Commit message: fix erc errors
Connections:
- C2 pad 2: GND -> Net-(J10-Pin_1)
- C3 pad 2: GND -> Net-(J10-Pin_1)
- C4 pad 2: GND -> Net-(J10-Pin_1)
- C5 pad 2: GND -> Net-(J10-Pin_1)
- J10 pad 1: GND -> Net-(J10-Pin_1)
- J11 pad 1: GND -> Net-(J10-Pin_1)
- J20 pad 18: Net-(J20-+5V) -> unconnected-(J20-+5V-Pad18)
- J23 pad 5: Net-(J18-SSRX-) -> Net-(J18-SSTX-)
- J23 pad 6: Net-(J18-SSRX+) -> Net-(J18-SSTX+)
- J23 pad 8: Net-(J18-SSTX-) -> Net-(J18-SSRX-)
- J23 pad 9: Net-(J18-SSTX+) -> Net-(J18-SSRX+)
- J24 pad 5: Net-(J22-SSRX-) -> Net-(J22-SSTX-)
- J24 pad 6: Net-(J22-SSRX+) -> Net-(J22-SSTX+)
- J24 pad 8: Net-(J22-SSTX-) -> Net-(J22-SSRX-)
- J24 pad 9: Net-(J22-SSTX+) -> Net-(J22-SSRX+)
- J25 pad 5: Net-(J21-SSRX-) -> Net-(J21-SSTX-)
- J25 pad 6: Net-(J21-SSRX+) -> Net-(J21-SSTX+)
- J25 pad 8: Net-(J21-SSTX-) -> Net-(J21-SSRX-)
- J25 pad 9: Net-(J21-SSTX+) -> Net-(J21-SSRX+)
- J27 pad 18: Net-(J20-+5V) -> unconnected-(J27-+5V-Pad18)
- J32 pad 5: Net-(J31-SSRX-) -> Net-(J31-SSTX-)
- J32 pad 6: Net-(J31-SSRX+) -> Net-(J31-SSTX+)
- J32 pad 8: Net-(J31-SSTX-) -> Net-(J31-SSRX-)
- J32 pad 9: Net-(J31-SSTX+) -> Net-(J31-SSRX+)
- J33 pad 9: GND -> Net-(J10-Pin_1)
- J5 pad 1: GND -> Net-(J10-Pin_1)
- J6 pad 1: GND -> Net-(J10-Pin_1)
- J7 pad 2: GND -> Net-(J10-Pin_1)
- J8 pad 1: GND -> Net-(J10-Pin_1)
- J9 pad 1: GND -> Net-(J10-Pin_1)
Changed lines of the file:
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@@
 	(net 160 "Net-(J20-CEC)")
 	(net 161 "Net-(J20-D0-)")
-	(net 162 "Net-(J20-+5V)")
+	(net 162 "Net-(J10-Pin_1)")
 	(net 163 "Net-(J20-CK+)")
 	(net 164 "Net-(J20-D1-)")
@@
 	(net 194 "Net-(J33-Pin_2)")
 	(net 195 "Net-(J33-Pin_1)")
+	(net 196 "unconnected-(J20-+5V-Pad18)")
+	(net 197 "unconnected-(J27-+5V-Pad18)")
 	(footprint "Connector_PinHeader_2.54mm:PinHeader_1x03_P2.54mm_Vertical"
 		(layer "F.Cu")
@@
 			(layers "F.Cu" "F.Mask" "F.Paste")
 			(roundrect_rratio 0.25)
-			(net 176 "Net-(J31-SSRX-)")
+			(net 191 "Net-(J31-SSTX-)")
 			(pinfunction "SSRX-")
 			(pintype "output")
@@
 			(layers "F.Cu" "F.Mask" "F.Paste")
 			(roundrect_rratio 0.25)
-			(net 192 "Net-(J31-SSRX+)")
+			(net 173 "Net-(J31-SSTX+)")
 			(pinfunction "SSRX+")
 			(pintype "output")
@@
 			(layers "F.Cu" "F.Mask" "F.Paste")
 			(roundrect_rratio 0.25)
-			(net 191 "Net-(J31-SSTX-)")
+			(net 176 "Net-(J31-SSRX-)")
 			(pinfunction "SSTX-")
 			(pintype "input")
@@
 			(layers "F.Cu" "F.Mask" "F.Paste")
 			(roundrect_rratio 0.25)
-			(net 173 "Net-(J31-SSTX+)")
+			(net 192 "Net-(J31-SSRX+)")
 			(pinfunction "SSTX+")
 			(pintype "input")
@@
 			(size 2.6 0.3)
 			(layers "F.Cu" "F.Mask" "F.Paste")
-			(net 162 "Net-(J20-+5V)")
+			(net 197 "unconnected-(J27-+5V-Pad18)")
 			(pinfunction "+5V")
-			(pintype "power_in")
+			(pintype "power_in+no_connect")
 		)
 		(pad "19" smd rect
@@
 			(layers "*.Cu" "*.Mask")
 			(remove_unused_layers no)
-			(net 96 "GND")
+			(net 162 "Net-(J10-Pin_1)")
 			(pintype "passive")
 		)
@@
 			(layers "F.Cu" "F.Mask" "F.Paste")
 			(roundrect_rratio 0.25)
-			(net 106 "Net-(J18-SSRX-)")
+			(net 107 "Net-(J18-SSTX-)")
 			(pinfunction "SSRX-")
 			(pintype "output")
@@
 			(layers "F.Cu" "F.Mask" "F.Paste")
 			(roundrect_rratio 0.25)
-			(net 150 "Net-(J18-SSRX+)")
+			(net 151 "Net-(J18-SSTX+)")
 			(pinfunction "SSRX+")
 			(pintype "output")
@@
 			(layers "F.Cu" "F.Mask" "F.Paste")
 			(roundrect_rratio 0.25)
-			(net 107 "Net-(J18-SSTX-)")
+			(net 106 "Net-(J18-SSRX-)")
 			(pinfunction "SSTX-")
 			(pintype "input")
@@
 			(layers "F.Cu" "F.Mask" "F.Paste")
 			(roundrect_rratio 0.25)
-			(net 151 "Net-(J18-SSTX+)")
+			(net 150 "Net-(J18-SSRX+)")
 			(pinfunction "SSTX+")
 			(pintype "input")
@@
 			(layers "*.Cu" "*.Mask")
 			(remove_unused_layers no)
-			(net 96 "GND")
+			(net 162 "Net-(J10-Pin_1)")
 			(pinfunction "Pin_1")
 			(pintype "passive")
@@
 			(layers "*.Cu" "*.Mask")
 			(remove_unused_layers no)
-			(net 96 "GND")
+			(net 162 "Net-(J10-Pin_1)")
 			(pinfunction "Pin_1")
 			(pintype "passive")
@@
 			(layers "*.Cu" "*.Mask")
 			(remove_unused_layers no)
-			(net 96 "GND")
+			(net 162 "Net-(J10-Pin_1)")
 			(pintype "passive")
 		)
@@
 			(layers "F.Cu" "F.Mask" "F.Paste")
 			(roundrect_rratio 0.25)
-			(net 186 "Net-(J22-SSRX-)")
+			(net 190 "Net-(J22-SSTX-)")
 			(pinfunction "SSRX-")
 			(pintype "output")
@@
 			(layers "F.Cu" "F.Mask" "F.Paste")
 			(roundrect_rratio 0.25)
-			(net 158 "Net-(J22-SSRX+)")
+			(net 157 "Net-(J22-SSTX+)")
 			(pinfunction "SSRX+")
 			(pintype "output")
@@
 			(layers "F.Cu" "F.Mask" "F.Paste")
 			(roundrect_rratio 0.25)
-			(net 190 "Net-(J22-SSTX-)")
+			(net 186 "Net-(J22-SSRX-)")
 			(pinfunction "SSTX-")
 			(pintype "input")
@@
 			(layers "F.Cu" "F.Mask" "F.Paste")
 			(roundrect_rratio 0.25)
-			(net 157 "Net-(J22-SSTX+)")
+			(net 158 "Net-(J22-SSRX+)")
 			(pinfunction "SSTX+")
 			(pintype "input")
@@
 			(layers "*.Cu" "*.Mask")
 			(remove_unused_layers no)
-			(net 96 "GND")
+			(net 162 "Net-(J10-Pin_1)")
 			(pinfunction "Pin_1")
 			(pintype "passive")
@@
 			(layers "*.Cu" "*.Mask")
 			(remove_unused_layers no)
-			(net 96 "GND")
+			(net 162 "Net-(J10-Pin_1)")
 			(pinfunction "Pin_9")
 			(pintype "passive")
@@
 			(net 26 "unconnected-(A1A-GND-Pad2)")
 			(pinfunction "GND")
-			(pintype "power_in")
+			(pintype "power_in+no_connect")
 		)
 		(pad "3" thru_hole circle
@@
 			(net 15 "unconnected-(A1A-GND-Pad4)")
 			(pinfunction "GND")
-			(pintype "power_in")
+			(pintype "power_in+no_connect")
 		)
 		(pad "5" thru_hole circle
@@
 			(net 49 "unconnected-(A1A-D5-Pad13)")
 			(pinfunction "D5")
-			(pintype "bidirectional")
+			(pintype "bidirectional+no_connect")
 		)
 		(pad "14" thru_hole circle
@@
 			(layers "*.Cu" "*.Mask")
 			(remove_unused_layers no)
-			(net 96 "GND")
+			(net 162 "Net-(J10-Pin_1)")
 			(pinfunction "Pin_1")
 			(pintype "passive")
@@
 			(layers "*.Cu" "*.Mask")
 			(remove_unused_layers no)
-			(net 96 "GND")
+			(net 162 "Net-(J10-Pin_1)")
 			(pintype "passive")
 		)
@@
 			(layers "*.Cu" "*.Mask")
 			(remove_unused_layers no)
-			(net 96 "GND")
+			(net 162 "Net-(J10-Pin_1)")
 			(pintype "passive")
 		)
@@
 			(layers "*.Cu" "*.Mask")
 			(remove_unused_layers no)
-			(net 96 "GND")
+			(net 162 "Net-(J10-Pin_1)")
 			(pinfunction "Pin_2")
 			(pintype "passive")
@@
 			(layers "*.Cu" "*.Mask")
 			(remove_unused_layers no)
-			(net 96 "GND")
+			(net 162 "Net-(J10-Pin_1)")
 			(pinfunction "Pin_1")
 			(pintype "passive")
@@
 			(layers "*.Cu" "*.Mask")
 			(remove_unused_layers no)
-			(net 96 "GND")
+			(net 162 "Net-(J10-Pin_1)")
 			(pinfunction "Pin_1")
 			(pintype "passive")
@@
 			(layers "F.Cu" "F.Mask" "F.Paste")
 			(roundrect_rratio 0.25)
-			(net 181 "Net-(J21-SSRX-)")
+			(net 185 "Net-(J21-SSTX-)")
 			(pinfunction "SSRX-")
 			(pintype "output")
@@
 			(layers "F.Cu" "F.Mask" "F.Paste")
 			(roundrect_rratio 0.25)
-			(net 183 "Net-(J21-SSRX+)")
+			(net 182 "Net-(J21-SSTX+)")
 			(pinfunction "SSRX+")
 			(pintype "output")
@@
 			(layers "F.Cu" "F.Mask" "F.Paste")
 			(roundrect_rratio 0.25)
-			(net 185 "Net-(J21-SSTX-)")
+			(net 181 "Net-(J21-SSRX-)")
 			(pinfunction "SSTX-")
 			(pintype "input")
@@
 			(layers "F.Cu" "F.Mask" "F.Paste")
 			(roundrect_rratio 0.25)
-			(net 182 "Net-(J21-SSTX+)")
+			(net 183 "Net-(J21-SSRX+)")
 			(pinfunction "SSTX+")
 			(pintype "input")
@@
 			(size 2.6 0.3)
 			(layers "F.Cu" "F.Mask" "F.Paste")
-			(net 162 "Net-(J20-+5V)")
+			(net 196 "unconnected-(J20-+5V-Pad18)")
 			(pinfunction "+5V")
-			(pintype "power_in")
+			(pintype "power_in+no_connect")
 		)
 		(pad "19" smd rect

Commit message: placement wip
Parts:
- added J29: HDMI_A, Connector_Video:HDMI_A_Molex_208658-1001_Horizontal, B.Cu at (272.5, 70.4)
- added J30: HDMI_A, Connector_Video:HDMI_A_Molex_208658-1001_Horizontal, F.Cu at (195.4, 40.0)
- A1, J18, J20, J24, J25: moved to B.Cu
- C2, C3, C4, C5: footprint Capacitor_THT:CP_Radial_D10.0mm_P5.00mm -> Capacitor_THT:CP_Radial_D8.0mm_P3.50mm
- moved S3 225.3 mm to (386.0, 27.3), turned to 180 degrees
- moved S2 208.6 mm to (383.3, 79.8)
- moved J26 168.9 mm to (361.7, 71.5)
- moved J28 168.9 mm to (361.7, 80.8)
- moved J31 159.0 mm to (379.4, 1.87)
- moved J32 159.0 mm to (397.1, 1.87)
- moved C5 157.8 mm to (265.0, 37.9)
- moved C4 156.1 mm to (265.0, 28.6)
- moved J6 150.8 mm to (255.2, 16.1)
- moved J8 150.6 mm to (259.4, 16.1)
- moved J10 150.6 mm to (268.3, 16.0)
- moved J9 150.5 mm to (263.8, 16.1)
- moved J11 150.5 mm to (272.8, 16.1)
- moved J12 150.4 mm to (277.4, 16.1)
- moved J5 150.0 mm to (251.0, 16.3)
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
Commit message: headphone jack
Parts:
- added J1: SJ1-3533NS, SJ1-3533NS:CUI_SJ1-3533NS, B.Cu at (264.0, 105.6)
- added J16: SJ1-3533NS, SJ1-3533NS:CUI_SJ1-3533NS, F.Cu at (251.7, 30.9)
- J28: moved to B.Cu
- moved J31 351.1 mm to (29.7, 32.7), turned to -90 degrees
- moved S3 349.7 mm to (55.3, 141.1)
- moved J26 342.1 mm to (24.6, 129.8), turned to -90 degrees
- moved J19 323.6 mm to (29.8, 51.2), turned to -90 degrees
- moved J32 317.5 mm to (81.4, 35.2), turned to 180 degrees
- moved J15 295.3 mm to (24.7, 145.0), turned to -90 degrees
- moved S2 281.2 mm to (108.8, 140.9), turned to 180 degrees
- moved J14 265.5 mm to (51.9, 29.9), turned to 180 degrees
- moved S1 264.2 mm to (81.2, 141.2), turned to 180 degrees
- moved J4 251.0 mm to (65.0, 30.0), turned to 180 degrees
- moved J17 235.7 mm to (98.6, 35.2), turned to 180 degrees
- moved J2 200.6 mm to (116.3, 35.3), turned to 180 degrees
- moved J5 139.1 mm to (222.0, 152.3), turned to 90 degrees
- moved J6 136.1 mm to (221.8, 148.1), turned to 90 degrees
- moved J8 133.2 mm to (221.8, 143.9), turned to 90 degrees
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
Commit message: routing
Parts:
- removed J1, J16: SJ1-3533NS, SJ1-3533NS:CUI_SJ1-3533NS
- removed J13: Conn_01x02_Pin, Connector_PinHeader_2.54mm:PinHeader_1x02_P2.54mm_Vertical
- removed J14, J15, J26, J28, J4: USB_C_Receptacle_PowerOnly_6P, Connector_USB:USB_C_Receptacle_GCT_USB4125-xx-x_6P_TopMnt_Horizontal
- removed J17, J18, J19, J2, J21, J22, J23, J24, J25, J31, J32: USB3_A, 692122030100:692122030100
- removed J20, J27, J29, J30: HDMI_A, Connector_Video:HDMI_A_Molex_208658-1001_Horizontal
- removed J3: Conn_01x03_Pin, Connector_PinHeader_2.54mm:PinHeader_1x03_P2.54mm_Vertical
- removed J34: Conn_02x05_Counter_Clockwise, Connector_PinHeader_2.54mm:PinHeader_2x05_P2.54mm_Vertical
- removed S1, S2, S3: RR511D1121, RR511D1121:E-SWITCH_RR511D1121
- added Camera1: USB3_A, 692122030100:692122030100, F.Cu at (84.0, 35.0)
- added Camera2: USB3_A, 692122030100:692122030100, B.Cu at (23.1, 71.3)
- added CentralFan1: Conn_01x02_Pin, Connector_PinHeader_2.54mm:PinHeader_1x02_P2.54mm_Vertical, F.Cu at (164.2, 143.1)
- added CentralLEDs1: Conn_01x03_Pin, Connector_PinHeader_2.54mm:PinHeader_1x03_P2.54mm_Vertical, F.Cu at (153.3, 143.1)
- added DisplayPWR1: USB3_A, 692122030100:692122030100, F.Cu at (155.2, 35.0)
- added DisplayPWR2: USB3_A, 692122030100:692122030100, F.Cu at (172.4, 35.0)
- added Display_A1: HDMI_A, Connector_Video:HDMI_A_Molex_208658-1001_Horizontal, B.Cu at (276.8, 67.1)
- added Display_A2: HDMI_A, Connector_Video:HDMI_A_Molex_208658-1001_Horizontal, F.Cu at (236.6, 34.3)
- added Display_B1: HDMI_A, Connector_Video:HDMI_A_Molex_208658-1001_Horizontal, B.Cu at (276.7, 87.2)
- added Display_B2: HDMI_A, Connector_Video:HDMI_A_Molex_208658-1001_Horizontal, F.Cu at (215.7, 34.3)
- added HeadFlat1: Conn_02x05_Counter_Clockwise, Connector_PinHeader_2.54mm:PinHeader_2x05_P2.54mm_Vertical, F.Cu at (196.9, 27.4)
- added MainPWR1: USB_C_Receptacle_PowerOnly_6P, Connector_USB:USB_C_Receptacle_GCT_USB4125-xx-x_6P_TopMnt_Horizontal, F.Cu at (28.1, 127.9)
- added MainPWR2: USB_C_Receptacle_PowerOnly_6P, Connector_USB:USB_C_Receptacle_GCT_USB4125-xx-x_6P_TopMnt_Horizontal, B.Cu at (279.0, 117.7)
- added Microphone1: USB3_A, 692122030100:692122030100, F.Cu at (101.7, 34.9)
- added Microphone2: USB3_A, 692122030100:692122030100, B.Cu at (23.0, 91.7)
- added Misc1: USB3_A, 692122030100:692122030100, F.Cu at (120.1, 34.9)
- added Misc2: USB3_A, 692122030100:692122030100, B.Cu at (23.1, 109.6)
- added Modem1: USB3_A, 692122030100:692122030100, F.Cu at (138.1, 34.9)
- added ModemPWR1: USB3_A, 692122030100:692122030100, F.Cu at (23.3, 36.5)
- added ON/OFFmain1: RR511D1121, RR511D1121:E-SWITCH_RR511D1121, F.Cu at (106.3, 140.4)
- added ON/OFFmodem1: RR511D1121, RR511D1121:E-SWITCH_RR511D1121, F.Cu at (79.8, 140.5)
- added ON/OFFperipherals1: RR511D1121, RR511D1121:E-SWITCH_RR511D1121, F.Cu at (53.7, 140.9)
- added PeripheralsPWR1: USB3_A, 692122030100:692122030100, F.Cu at (23.3, 54.2)
- added RechargeA1: USB_C_Receptacle_PowerOnly_6P, Connector_USB:USB_C_Receptacle_GCT_USB4125-xx-x_6P_TopMnt_Horizontal, F.Cu at (47.0, 29.9)
- added RechargeB1: USB_C_Receptacle_PowerOnly_6P, Connector_USB:USB_C_Receptacle_GCT_USB4125-xx-x_6P_TopMnt_Horizontal, F.Cu at (62.9, 29.9)
- added RechargeB2: USB_C_Receptacle_PowerOnly_6P, Connector_USB:USB_C_Receptacle_GCT_USB4125-xx-x_6P_TopMnt_Horizontal, F.Cu at (28.0, 141.6)
- added Speaker1: SJ1-3533NS, SJ1-3533NS:CUI_SJ1-3533NS, F.Cu at (256.4, 31.0)
- added Speaker2: SJ1-3533NS, SJ1-3533NS:CUI_SJ1-3533NS, B.Cu at (269.8, 104.7)
- moved R1 12.7 mm to (152.5, 137.6), turned to 0 degrees
- moved J33 11.5 mm to (251.8, 141.7), turned to 0 degrees
- moved C1 4.06 mm to (143.4, 143.1), turned to 90 degrees
- moved J7 2.90 mm to (229.4, 143.0)
- moved C5 2.88 mm to (240.7, 138.6)
- moved C3 2.88 mm to (240.7, 129.8)
- moved C4 2.88 mm to (231.4, 138.6)
- moved C2 2.88 mm to (231.3, 129.8)
- moved R3 2.88 mm to (254.1, 138.1)
- moved J6 2.84 mm to (219.0, 148.6)
- moved J12 2.81 mm to (219.0, 125.6)
- moved J9 2.80 mm to (219.0, 139.4)
- moved J8 2.80 mm to (219.0, 144.0)
- moved J11 2.75 mm to (219.0, 130.2)
- moved J10 2.71 mm to (219.0, 134.8)
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Routing:
- net GND: track 0.00 -> 865.6 mm, vias 0 -> 17
- net Net-(MainPWR1-SHIELD): track 0.00 -> 409.7 mm
- net Net-(MainPWR1-CC2): track 0.00 -> 354.2 mm, vias 0 -> 3
- net Net-(MainPWR1-CC1): track 0.00 -> 340.7 mm, vias 0 -> 3
- net /Power Distribution/+5V peripherals: track 0.00 -> 279.2 mm, vias 0 -> 2
- net Net-(MainPWR1-VBUS-PadA9): track 0.00 -> 200.7 mm, vias 0 -> 3
- net Net-(MainPWR2-VBUS-PadA9): track 0.00 -> 192.7 mm, vias 0 -> 2
- net Net-(Misc1-SHIELD): track 0.00 -> 188.5 mm, vias 0 -> 1
- net Net-(DisplayPWR1-SHIELD): track 0.00 -> 186.9 mm
- net Net-(Misc1-SSTX-): track 0.00 -> 177.3 mm, vias 0 -> 1
- net Net-(Misc1-SSTX+): track 0.00 -> 175.4 mm, vias 0 -> 1
- net Net-(Misc1-D-): track 0.00 -> 165.5 mm, vias 0 -> 1
- net Net-(Misc1-SSRX-): track 0.00 -> 165.4 mm, vias 0 -> 3
- net Net-(Misc1-D+): track 0.00 -> 163.6 mm, vias 0 -> 3
- net Net-(Misc1-VBUS): track 0.00 -> 161.2 mm, vias 0 -> 1
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Other:
- board outline added: 273.4 x 131.6 mm

Commit message: Update DYNAMO-PCB.kicad_pcb
Parts:
- moved HeadFlat1 83.6 mm to (113.3, 27.0)
- moved Modem1 52.2 mm to (85.9, 34.8)
- moved Microphone1 47.5 mm to (149.2, 34.8)
- moved Misc1 47.3 mm to (167.4, 34.8)
- moved Camera1 47.1 mm to (131.1, 34.9)
- moved DisplayPWR2 32.2 mm to (204.6, 34.7)
- moved DisplayPWR1 30.7 mm to (185.9, 34.7)
- moved Display_A2 12.6 mm to (249.2, 33.8)
- moved Display_B2 11.7 mm to (227.3, 33.8)
- moved Speaker1 11.5 mm to (267.9, 30.8)
- moved RechargeB2 9.49 mm to (19.1, 145.0)
- moved MainPWR1 9.49 mm to (19.2, 131.4)
- moved ModemPWR1 6.00 mm to (23.2, 42.5)
- moved PeripheralsPWR1 6.00 mm to (23.2, 60.2)
- moved Camera2 5.90 mm to (23.1, 77.2)
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Routing:
- net Net-(Modem1-SSRX-): track 135.7 -> 50.5 mm, vias 2 -> 0
- net Net-(Misc1-SSTX-): track 177.3 -> 260.3 mm
- net Net-(Misc1-VBUS): track 161.2 -> 232.9 mm
- net Net-(Microphone1-D+): track 128.9 -> 198.7 mm, vias 1 -> 5
- net Net-(Modem1-SHIELD): track 151.9 -> 84.5 mm
- net Net-(Misc1-DRAIN): track 159.7 -> 222.9 mm, vias 1 -> 3
- net Net-(Modem1-SSTX-): track 121.0 -> 59.3 mm, vias 4 -> 0
- net Net-(Microphone1-SSRX+): track 129.6 -> 191.0 mm, vias 3 -> 5
- net Net-(Microphone1-SHIELD): track 145.7 -> 206.9 mm, vias 1 -> 2
- net Net-(Misc1-SSRX+): track 152.8 -> 213.5 mm, vias 1 -> 5
- net Net-(Modem1-SSRX+): track 114.0 -> 54.7 mm, vias 2 -> 0
- net Net-(Modem1-DRAIN): track 116.8 -> 57.9 mm
- net Net-(Modem1-D+): track 113.7 -> 55.1 mm, vias 4 -> 0
- net Net-(Camera1-D+): track 93.3 -> 151.0 mm, vias 3 -> 1
- net /Power Distribution/+5V peripherals: track 279.2 -> 336.4 mm, vias 2 -> 1
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Other:
- outline, holes or cut-outs redrawn

Commit message: further simplified
Parts:
- removed Camera1, Camera2, Microphone1, Microphone2, Misc1, Misc2: USB3_A, 692122030100:692122030100
- removed Display_A1, Display_A2, Display_B1, Display_B2: HDMI_A, Connector_Video:HDMI_A_Molex_208658-1001_Horizontal
- removed Speaker1, Speaker2: SJ1-3533NS, SJ1-3533NS:CUI_SJ1-3533NS
- MainPWR2: moved to F.Cu
- moved MainPWR2 126.5 mm to (154.9, 142.1)
- moved CentralFan1 105.9 mm to (81.5, 77.0), turned to 180 degrees
- moved R1 90.9 mm to (76.0, 88.6), turned to 90 degrees
- moved CentralLEDs1 90.6 mm to (81.5, 87.8), turned to 180 degrees
- moved C1 76.8 mm to (81.5, 97.7), turned to 180 degrees
- moved R3 70.8 mm to (234.4, 70.0), turned to 180 degrees
- moved J33 70.7 mm to (238.0, 72.3), turned to 90 degrees
- moved R2 65.5 mm to (234.3, 74.4), turned to 180 degrees
- moved J5 56.8 mm to (248.7, 102.5), turned to 180 degrees
- moved C5 55.5 mm to (234.9, 83.4), turned to 180 degrees
- moved J6 50.6 mm to (244.9, 105.1), turned to 180 degrees
- moved J7 49.3 mm to (239.3, 94.7), turned to 180 degrees
- moved C3 48.6 mm to (226.1, 83.4), turned to 180 degrees
- moved C4 46.0 mm to (234.9, 92.7), turned to 180 degrees
- moved MainPWR1 45.4 mm to (49.8, 97.8)
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Routing:
- net GND: track 896.6 -> 448.2 mm, vias 13 -> 3
- net Net-(Misc1-SSTX-): track 260.3 -> 0.00 mm, vias 1 -> 0
- net Net-(Misc1-VBUS): track 232.9 -> 0.00 mm, vias 1 -> 0
- net Net-(Misc1-DRAIN): track 222.9 -> 0.00 mm, vias 3 -> 0
- net Net-(Misc1-SHIELD): track 221.5 -> 0.00 mm, vias 2 -> 0
- net Net-(Misc1-D-): track 217.8 -> 0.00 mm, vias 3 -> 0
- net Net-(Misc1-SSTX+): track 216.9 -> 0.00 mm, vias 1 -> 0
- net Net-(Misc1-D+): track 215.1 -> 0.00 mm, vias 1 -> 0
- net Net-(Misc1-SSRX+): track 213.5 -> 0.00 mm, vias 5 -> 0
- net Net-(Misc1-SSRX-): track 212.6 -> 0.00 mm, vias 3 -> 0
- net Net-(Microphone1-SHIELD): track 206.9 -> 0.00 mm, vias 2 -> 0
- net Net-(Microphone1-SSTX+): track 202.4 -> 0.00 mm, vias 3 -> 0
- net Net-(Microphone1-D+): track 198.7 -> 0.00 mm, vias 5 -> 0
- net Net-(Microphone1-SSTX-): track 193.9 -> 0.00 mm, vias 3 -> 0
- net Net-(Microphone1-SSRX+): track 191.0 -> 0.00 mm, vias 5 -> 0
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Other:
- board size 273.4 x 131.6 mm -> 208.9 x 129.5 mm
